File: stm32h755.kicad_sch (KiCad schematic)
At the start: 29 parts, among them U1 STM32H757IITx

Commit message: Decoupling Capacitors Placed
Parts:
- C19, C20, C21: footprint Capacitor_SMD:C_01005_0402Metric -> Capacitor_SMD:C_0201_0603Metric
- C22, C23, C24, C27, C28: footprint (none) -> Capacitor_SMD:C_0201_0603Metric
- C25, C26: footprint (none) -> Capacitor_SMD:C_01005_0402Metric
Connections:
- net +3.3VA: no longer C1.1, C10.1, C11.1, C12.1, C13.1, C14.1, C15.1, C16.1, C17.1, C2.1, C25.1, C28.1, C3.1, C4.1, C5.1, C6.1, C7.1, C8.1, C9.1, U1.113 (VDD), U1.120 (VDD50_USB), U1.121 (VDD33_USB), U1.126 (VDD), U1.13 (VDD), U1.136 (VDD), U1.152 (VDD), U1.160 (VDD), U1.176 (VDD), U1.25 (VDD), U1.44 (VDD), U1.48 (VDD), U1.65 (VDD), U1.7 (VDD), U1.71 (VDD), U1.84 (VDD), U1.92 (VDD), U1.99 (VDD)
- new net +3V3: C1.1, C10.1, C11.1, C12.1, C13.1, C14.1, C15.1, C16.1, C17.1, C2.1, C25.1, C28.1, C3.1, C4.1, C5.1, C6.1, C7.1, C8.1, C9.1, U1.113 (VDD), U1.120 (VDD50_USB), U1.121 (VDD33_USB), U1.126 (VDD), U1.13 (VDD), U1.136 (VDD), U1.152 (VDD), U1.160 (VDD), U1.176 (VDD), U1.25 (VDD), U1.44 (VDD), U1.48 (VDD), U1.65 (VDD), U1.7 (VDD), U1.71 (VDD), U1.84 (VDD), U1.92 (VDD), U1.99 (VDD)
Changed lines of the file:
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@@
 			)
 		)
-		(property "Footprint" ""
+		(property "Footprint" "Capacitor_SMD:C_0201_0603Metric"
 			(at 244.8052 394.97 0)
 			(effects
@@
 			)
 		)
-		(property "Footprint" ""
+		(property "Footprint" "Capacitor_SMD:C_0201_0603Metric"
 			(at 36.5252 365.76 0)
 			(effects
@@
 			)
 		)
-		(property "Footprint" ""
+		(property "Footprint" "Capacitor_SMD:C_01005_0402Metric"
 			(at 346.4052 394.97 0)
 			(effects
@@
 			)
 		)
-		(property "Footprint" "Capacitor_SMD:C_01005_0402Metric"
+		(property "Footprint" "Capacitor_SMD:C_0201_0603Metric"
 			(at 322.2752 396.24 0)
 			(effects
@@
 			)
 		)
-		(property "Footprint" ""
+		(property "Footprint" "Capacitor_SMD:C_0201_0603Metric"
 			(at 359.1052 394.97 0)
 			(effects
@@
 			)
 		)
-		(property "Footprint" "Capacitor_SMD:C_01005_0402Metric"
+		(property "Footprint" "Capacitor_SMD:C_0201_0603Metric"
 			(at 300.6852 396.24 0)
 			(effects
@@
 			)
 		)
-		(property "Footprint" "Capacitor_SMD:C_01005_0402Metric"
+		(property "Footprint" "Capacitor_SMD:C_0201_0603Metric"
 			(at 312.1152 396.24 0)
 			(effects
@@
 	)
 	(symbol
-		(lib_id "power:+3V3")
-		(at 361.95 386.08 270)
-		(unit 1)
-		(exclude_from_sim no)
-		(in_bom yes)
-		(on_board yes)
-		(dnp no)
-		(fields_autoplaced yes)
-		(property "Reference" "#PWR011"
-			(at 358.14 386.08 0)
-			(effects
-				(font
-					(size 1.27 1.27)
-				)
-				(hide yes)
-			)
-		)
-		(property "Value" "+3V3"
-			(at 365.76 386.0799 90)
-			(effects
-				(font
-					(size 1.27 1.27)
-				)
-				(justify left)
-			)
-		)
-		(property "Footprint" ""
-			(at 361.95 386.08 0)
-			(effects
-				(font
-					(size 1.27 1.27)
-				)
-				(hide yes)
-			)
-		)
-		(property "Datasheet" ""
-			(at 361.95 386.08 0)
-			(effects
-				(font
-					(size 1.27 1.27)
-				)
-				(hide yes)
-			)
-		)
-		(property "Description" "Power symbol creates a global label with name \"+3V3\""
-			(at 361.95 386.08 0)
-			(effects
-				(font
-					(size 1.27 1.27)
-				)
-				(hide yes)
-			)
-		)
-		(pin "1"
-		)
-		(instances
-			(project "stm32h755"
-				(path "/63df81d5-7d5d-484c-b8b8-55609d33e66e"
-					(reference "#PWR011")
-					(unit 1)
-				)
-			)
-		)
-	)
-	(symbol
 		(lib_id "Device:C")
 		(at 255.27 391.16 0)
@@
 			)
 		)
-		(property "Footprint" ""
+		(property "Footprint" "Capacitor_SMD:C_0201_0603Metric"
 			(at 256.2352 394.97 0)
 			(effects
@@
 			)
 		)
-		(property "Footprint" ""
+		(property "Footprint" "Capacitor_SMD:C_01005_0402Metric"
 			(at 23.8252 365.76 0)
 			(effects
@@
 			)
 		)
-		(property "Footprint" ""
+		(property "Footprint" "Capacitor_SMD:C_0201_0603Metric"
 			(at 266.3952 394.97 0)
 			(effects

Commit message: Redesigned PCB
Parts:
- added C29: 100nF, Capacitor_SMD:C_01005_0402Metric, symbol Device:C
- added C30: 1uF, Capacitor_SMD:C_0201_0603Metric, symbol Device:C
- added C31, C32: 10uF, Capacitor_SMD:C_0603_1608Metric, symbol Device:C
- added U2: AMS1117, Package_TO_SOT_SMD:SOT-223-3_TabPin2, symbol Regulator_Linear:AMS1117
Connections:
- net +3V3 is gone; now on net +3.3VA: C1.1, C10.1, C11.1, C12.1, C13.1, C14.1, C15.1, C16.1, C17.1, C2.1, C25.1, C28.1, C3.1, C4.1, C5.1, C6.1, C7.1, C8.1, C9.1, U1.113 (VDD), U1.120 (VDD50_USB), U1.121 (VDD33_USB), U1.126 (VDD), U1.13 (VDD), U1.136 (VDD), U1.152 (VDD), U1.160 (VDD), U1.176 (VDD), U1.25 (VDD), U1.44 (VDD), U1.48 (VDD), U1.65 (VDD), U1.7 (VDD), U1.71 (VDD), U1.84 (VDD), U1.92 (VDD), U1.99 (VDD)
- net VDDLDO is gone; now on net +3.3VA: C22.1, C23.1, C24.1, U1.135 (VDDLDO), U1.175 (VDDLDO), U1.82 (VDDLDO)
- net +3.3VA: now also U1.39 (VREF+), C29.1, C30.1, C31.1, U2.2 (VO)
- net GND: now also C29.2, C30.2, C31.2, C32.2, U2.1 (ADJ)
- new net VIN: C32.1, U2.3 (VI)
- no-connect marks 3 -> 7

Commit message: Redesigned PCB
Parts:
- added D1: LED, LED_SMD:LED_0201_0603Metric, symbol Device:LED
- added J1, J2, J3, J4: Conn_01x04_Pin, Connector_PinHeader_2.54mm:PinHeader_1x04_P2.54mm_Horizontal, symbol Connector:Conn_01x04_Pin
- added J5: Conn_01x08_Pin, Connector_PinHeader_2.54mm:PinHeader_1x08_P2.54mm_Vertical, symbol Connector:Conn_01x08_Pin
- added J6: Conn_01x02_Pin, Connector_PinHeader_2.54mm:PinHeader_1x02_P2.54mm_Vertical, symbol Connector:Conn_01x02_Pin
- added R1: 10K, Resistor_SMD:R_0201_0603Metric, symbol Device:R
- added R2: R, Resistor_SMD:R_0201_0603Metric, symbol Device:R
Connections:
- net GND: now also D1.1 (K), J1.1 (Pin_1), J2.1 (Pin_1), J3.1 (Pin_1), J4.1 (Pin_1), J6.1 (Pin_1), R2.2
- net at U1.132 (PA13): now also J1.3 (Pin_3)
- net at U1.138 (PA14): now also J1.2 (Pin_2)
- net at U1.143 (PD0): now also J5.1 (Pin_1)
- net at U1.144 (PD1): now also J5.2 (Pin_2)
- net at U1.145 (PD2): now also J5.3 (Pin_3)
- net at U1.146 (PD3): now also J5.4 (Pin_4)
- net at U1.147 (PD4): now also J5.5 (Pin_5)
- net at U1.148 (PD5): now also J5.6 (Pin_6)
- net at U1.149 (PD6): now also J5.7 (Pin_7)
- net at U1.150 (PD7): now also J5.8 (Pin_8)
- net at U1.165 (PB6): now also J4.3 (Pin_3)
- net at U1.166 (PB7): now also J4.2 (Pin_2)
- net at U1.167 (BOOT0): now also R2.1
- net at U1.43 (PA2): now also J2.3 (Pin_3)
- net at U1.46 (PA3): now also J2.2 (Pin_2)
- net at U1.87 (PB14): now also J3.3 (Pin_3)
- net at U1.88 (PB15): now also J3.2 (Pin_2)
- net +3.3VA renamed +3V3
- net +3V3: now also J1.4 (Pin_4), J2.4 (Pin_4), J3.4 (Pin_4), J4.4 (Pin_4), R1.2; no longer C29.1, C30.1, U1.39 (VREF+)
- removed net VCAP: C18.1, C19.1, C20.1, C21.1, U1.101 (VCAPDSI), U1.133 (VCAP), U1.172 (VCAP), U1.80 (VCAP)
- net VIN renamed +5V
- net +5V: now also J6.2 (Pin_2)
- new net: C18.1, U1.101 (VCAPDSI)
- new net: C21.1, U1.133 (VCAP)
- new net: C20.1, U1.172 (VCAP)
- new net: C19.1, U1.80 (VCAP)
- new net: D1.2 (A), R1.1
- new net VREF: C29.1, C30.1, U1.39 (VREF+)
- no-connect marks 7 -> 110
Other:
- moved on the sheet: C18, C19, C20, C21, C22, C23, C24, C25, C28, C32
